Commit message: Tweak robot dimensions

File: description/robot_core.xacro (robot description, xacro)
@@ -23,18 +23,18 @@
   <link name="chassis">
     <visual>
-      <origin xyz="0.15 0 0.075"/>
+      <origin xyz="0.16 0 0.032"/>
       <geometry>
-        <box size="0.3 0.3 0.15"/>
+        <box size="0.25 0.2 0.07"/>
       </geometry>
       <material name="white"/>
     </visual>
     <collision>
-      <origin xyz="0.15 0 0.075"/>
+      <origin xyz="0.16 0 0.032"/>
       <geometry>
-        <box size="0.3 0.3 0.15"/>
+        <box size="0.25 0.2 0.07"/>
       </geometry>
     </collision>
-    <xacro:inertial_box mass="0.5" x="0.3" y="0.3" z="0.15">
-      <origin xyz="0.15 0 0.075" rpy="0 0 0" />
+    <xacro:inertial_box mass="0.5" x="0.25" y="0.2" z="0.07">
+      <origin xyz="0.16 0 0.032" rpy="0 0 0" />
     </xacro:inertial_box>
   </link>
@@ -45,5 +45,5 @@
     <parent link="base_link"/>
     <child link="left_wheel"/>
-    <origin xyz="0 0.175 0" rpy="-${pi/2} 0 0"/>
+    <origin xyz="0 0.11 -0.02" rpy="-${pi/2} 0 0"/>
     <axis xyz="0 0 1" />
   </joint>
@@ -51,5 +51,5 @@
     <visual>
       <geometry>
-        <cylinder radius="0.05" length="0.04"/>
+        <cylinder radius="0.035" length="0.028"/>
       </geometry>
       <material name="blue"/>
@@ -57,8 +57,8 @@
     <collision>
       <geometry>
-        <cylinder radius="0.05" length="0.04"/>
+        <sphere radius="0.035"/>
       </geometry>
     </collision>
-    <xacro:inertial_cylinder mass="0.1" length="0.04" radius="0.05">
+    <xacro:inertial_cylinder mass="0.1" length="0.028" radius="0.035">
       <origin xyz="0 0 0" rpy="0 0 0" />
     </xacro:inertial_cylinder>
@@ -70,5 +70,5 @@
     <parent link="base_link"/>
     <child link="right_wheel"/>
-    <origin xyz="0 -0.175 0" rpy="${pi/2} 0 0"/>
+    <origin xyz="0 -0.11 -0.02" rpy="${pi/2} 0 0"/>
     <axis xyz="0 0 -1" />
   </joint>
@@ -76,5 +76,5 @@
     <visual>
       <geometry>
-        <cylinder radius="0.05" length="0.04"/>
+        <cylinder radius="0.035" length="0.028"/>
       </geometry>
       <material name="blue"/>
@@ -82,8 +82,8 @@
     <collision>
       <geometry>
-        <cylinder radius="0.05" length="0.04"/>
+        <sphere radius="0.035"/>
       </geometry>
     </collision>
-    <xacro:inertial_cylinder mass="0.1" length="0.04" radius="0.05">
+    <xacro:inertial_cylinder mass="0.1" length="0.028" radius="0.035">
       <origin xyz="0 0 0" rpy="0 0 0" />
     </xacro:inertial_cylinder>
