Commit message: Add gezebo support

File: description/robot.urdf.xacro (robot description, xacro)
@@ -2,3 +2,4 @@
 <robot xmlns:xacro="http://www.ros.org/wiki/xacro"  name="robot">
   <xacro:include filename="robot_core.xacro"/>
+  <xacro:include filename="gazebo_control.xacro"/>
 </robot>

File: description/robot_core.xacro (robot description, xacro)
@@ -1,4 +1,4 @@
 <?xml version="1.0"?>
-<robot xmlns:xacro="http://www.ros.org/wiki/xacro"  name="robot">
+<robot xmlns:xacro="http://www.ros.org/wiki/xacro">
   <xacro:include filename="inertial_macros.xacro"/>
   <material name="white">
@@ -16,5 +16,5 @@
   <link name="base_link">
   </link>
-  <joint name="classis_joint" type="fixed">
+  <joint name="chassis_joint" type="fixed">
     <parent link="base_link"/>
     <child link="chassis"/>
@@ -39,4 +39,7 @@
     </xacro:inertial_box>
   </link>
+  <gazebo reference="chassis">
+    <material>Gazebo/White</material>
+  </gazebo>
   <joint name="left_wheel_joint" type="continuous">
     <parent link="base_link"/>
@@ -47,5 +50,4 @@
   <link name="left_wheel">
     <visual>
-      <origin xyz="0 0 0"/>
       <geometry>
         <cylinder radius="0.05" length="0.04"/>
@@ -54,5 +56,4 @@
     </visual>
     <collision>
-      <origin xyz="0 0 0"/>
       <geometry>
         <cylinder radius="0.05" length="0.04"/>
@@ -63,13 +64,15 @@
     </xacro:inertial_cylinder>
   </link>
+  <gazebo reference="left_wheel">
+    <material>Gazebo/Blue</material>
+  </gazebo>
   <joint name="right_wheel_joint" type="continuous">
     <parent link="base_link"/>
     <child link="right_wheel"/>
     <origin xyz="0 -0.175 0" rpy="${pi/2} 0 0"/>
-    <axis xyz="0 0 1" />
+    <axis xyz="0 0 -1" />
   </joint>
   <link name="right_wheel">
     <visual>
-      <origin xyz="0 0 0"/>
       <geometry>
         <cylinder radius="0.05" length="0.04"/>
@@ -78,5 +81,4 @@
     </visual>
     <collision>
-      <origin xyz="0 0 0"/>
       <geometry>
         <cylinder radius="0.05" length="0.04"/>
@@ -87,4 +89,7 @@
     </xacro:inertial_cylinder>
   </link>
+  <gazebo reference="right_wheel">
+    <material>Gazebo/Blue</material>
+  </gazebo>
   <joint name="caster_wheel_joint" type="fixed">
     <parent link="chassis"/>
@@ -108,3 +113,8 @@
     </xacro:inertial_sphere>
   </link>
+<gazebo reference="caster_wheel">
+    <material>Gazebo/Black</material>
+    <mu1 value="0.001"/>
+    <mu2 value="0.001"/>
+</gazebo>
 </robot>

Commit message: Add robot launch script

File: description/robot.urdf.xacro (robot description, xacro)
@@ -2,4 +2,5 @@
 <robot xmlns:xacro="http://www.ros.org/wiki/xacro"  name="robot">
   <xacro:arg name="use_ros2_control" default="true"/>
+  <xacro:arg name="sim_mode" default="false"/>
   <xacro:include filename="robot_core.xacro"/>
   <!-- <xacro:include filename="gazebo_control.xacro" /> -->

File: description/ros2_control.xacro (robot description, xacro)
@@ -1,9 +1,48 @@
 <?xml version="1.0"?>
 <robot xmlns:xacro="http://www.ros.org/wiki/xacro">
-  <ros2_control name="GazeboSystem" type="system">
-    <hardware>
-        <plugin>gazebo_ros2_control/GazeboSystem</plugin>
-    </hardware>
-    <joint name="left_wheel_joint">
+  <xacro:unless value="$(arg sim_mode)">
+      <ros2_control name="RealRobot" type="system">
+          <hardware>
+              <plugin>diffdrive_arduino/DiffDriveArduino</plugin>
+              <param name="left_wheel_name">left_wheel_joint</param>
+              <param name="right_wheel_name">right_wheel_joint</param>
+              <param name="loop_rate">30</param>
+              <param name="device">/dev/ttyUSB0</param>
+              <param name="baud_rate">57600</param>
+              <param name="timeout">1000</param>
+              <param name="enc_counts_per_rev">3436</param>
+          </hardware>
+          <joint name="left_wheel_joint">
+              <command_interface name="velocity">
+                  <param name="min">-10</param>
+                  <param name="max">10</param>
+              </command_interface>
+              <state_interface name="velocity"/>
+              <state_interface name="position"/>
+          </joint>
+          <joint name="right_wheel_joint">
+              <command_interface name="velocity">
+                  <param name="min">-10</param>
+                  <param name="max">10</param>
+              </command_interface>
+              <state_interface name="velocity"/>
+              <state_interface name="position"/>
+          </joint>
+      </ros2_control>
+  </xacro:unless>
+  <xacro:if value="$(arg sim_mode)">
+    <ros2_control name="GazeboSystem" type="system">
+      <hardware>
+          <plugin>gazebo_ros2_control/GazeboSystem</plugin>
+      </hardware>
+      <joint name="left_wheel_joint">
+          <command_interface name="velocity">
+            <param name="min">-10</param>
+            <param name="max">10</param>
+          </command_interface>
+          <state_interface name="velocity"/>
+          <state_interface name="position"/>
+      </joint>
+      <joint name="right_wheel_joint">
         <command_interface name="velocity">
           <param name="min">-10</param>
@@ -12,18 +51,12 @@
         <state_interface name="velocity"/>
         <state_interface name="position"/>
-    </joint>
-    <joint name="right_wheel_joint">
-      <command_interface name="velocity">
-        <param name="min">-10</param>
-        <param name="max">10</param>
-      </command_interface>
-      <state_interface name="velocity"/>
-      <state_interface name="position"/>
-    </joint>
-  </ros2_control>
-  <gazebo>
-    <plugin name="gazebo_ros2_control" filename="libgazebo_ros2_control.so">
-        <parameters>$(find lawnbot_proto)/config/my_controllers.yaml</parameters>
-    </plugin>
-  </gazebo>
+      </joint>
+    </ros2_control>
+    <gazebo>
+      <plugin name="gazebo_ros2_control" filename="libgazebo_ros2_control.so">
+          <parameters>$(find lawnbot_proto)/config/my_controllers.yaml</parameters>
+          <!-- <parameters>$(find lawnbot_proto)/config/gaz_ros2_ctl_use_sim.yaml</parameters> -->
+      </plugin>
+    </gazebo>
+  </xacro:if>
 </robot>
